Commit message: added collitions to urdfs and changes in simulation

File: modelos/manipuladores/katana/football_pitch.urdf (robot description, URDF)
Before this commit: robot football_pitch.urdf, 1 links, 0 joints
Links:
- link football_pitch: geometry collision box size=0.5 0.65 0.02; visual mesh filename=package://katana/katana/Football+Pitch.stl scale=0.003 0.003 0.003

File: modelos/manipuladores/katana/katana.urdf (robot description, URDF)
Before this commit: robot katana_300_6m180, 11 links, 10 joints
Links:
- link katana_l_finger_link: geometry collision box size=0.03 0.005 0.02; visual mesh filename=package://katana/katana/katana_gripper_l_finger.stl
- link katana_r_finger_link: geometry collision box size=0.03 0.005 0.02; visual mesh filename=package://katana/katana/katana_gripper_r_finger.stl
Joints:
- joint katana_motor4_lift_joint: origin xyz=0.139 0 0 rpy=$1.5708 0 0 -> xyz=0.139 0 0 rpy=1.5708 0 0
