Commit message: added models and updated simulation for katana

File: modelos/manipuladores/katana/katana.urdf (robot description, URDF)
Before this commit: robot katana_300_6m180, 11 links, 10 joints
Joints:
- joint katana_motor3_lift_joint: axis 0 0 1 -> 0 1 0
- joint katana_motor4_lift_joint: axis 0 0 1 -> 0 1 0

Commit message: se agrega código de pick and place (arreglar aun)

File: modelos/manipuladores/katana/katana.urdf (robot description, URDF)
Before this commit: robot katana_300_6m180, 11 links, 10 joints
Links:
- link katana_l_finger_link: geometry collision box size=0.02 0.005 0.02; collision box size=0.05 0.005 0.02
- link katana_r_finger_link: geometry collision box size=0.02 0.005 0.02; collision box size=0.05 0.005 0.02
