Commit message: try to collide bag and end effector

File: modelos/manipuladores/brazo_omni_description/urdf/brazo_omni.xacro (robot description, xacro)
@@ -84,5 +84,5 @@
   </collision>
 </link>
-<link name="end_effector_1">
+<link name="end_effector_1" concave="yes">
   <inertial>
     <origin xyz="0.0018769943609454375 -0.02500000000000892 0.007657259532162564" rpy="0 0 0"/>
@@ -97,5 +97,5 @@
     <material name="silver"/>
   </visual>
-  <collision>
+  <collision >
     <origin xyz="-0.0 -0.025 -0.475" rpy="0 0 0"/>
     <geometry>

File: modelos/objetos/mini_bag_description/urdf/mini_bag.xacro (robot description, xacro)
@@ -17,5 +17,5 @@
     <material name="silver"/>
   </visual>
-  <collision>
+  <collision concave="yes">
     <origin xyz="0 0 0" rpy="0 0 0"/>
     <geometry>
