Commit message: collision ready

File: modelos/manipuladores/brazo_omni_v2_description/urdf/brazo_omni_v2.xacro (robot description, xacro)
@@ -124,5 +124,5 @@
   </collision>
 </link>
-<link name="l2_1">
+<!-- <link name="l2_1">
   <inertial>
     <origin xyz="1.592451013345226e-10 -0.024999988944218367 0.06944981476509296" rpy="0 0 0"/>
@@ -143,6 +143,6 @@
     </geometry>
   </collision>
-</link>
-<link name="l3_1">
+</link> -->
+<!-- <link name="l3_1">
   <inertial>
     <origin xyz="1.5924509514741469e-10 -0.024999988944218378 0.06944981476509277" rpy="0 0 0"/>
@@ -163,5 +163,6 @@
     </geometry>
   </collision>
-</link>
+</link>  -->
+<!--
 <link name="eff_1_1">
   <inertial>
@@ -183,5 +184,5 @@
     </geometry>
   </collision>
-</link>
+</link> -->
 <joint name="l1_to_base_link" type="revolute">
   <origin xyz="0.0 0.025 0.025" rpy="0 0 0"/>
@@ -217,5 +218,6 @@
   <child link="eff_2_1"/>
 </joint>
-<joint name="Revoluci�n 6" type="revolute">
+<!--
+<joint name="Revolucion 6" type="revolute">
   <origin xyz="0.0 0.0 0.15" rpy="0 0 0"/>
   <parent link="l1_1"/>
@@ -224,5 +226,5 @@
   <limit upper="1.989675" lower="-1.989675" effort="100" velocity="100"/>
 </joint>
-<joint name="Revoluci�n 7" type="revolute">
+<joint name="Revolucion 7" type="revolute">
   <origin xyz="0.0 0.0 0.15" rpy="0 0 0"/>
   <parent link="l2_1"/>
@@ -231,5 +233,5 @@
   <limit upper="1.989675" lower="-1.989675" effort="100" velocity="100"/>
 </joint>
-<joint name="Revoluci�n 8" type="revolute">
+<joint name="Revolucion 8" type="revolute">
   <origin xyz="0.0 0.0 0.15" rpy="0 0 0"/>
   <parent link="l3_1"/>
@@ -237,4 +239,4 @@
   <axis xyz="-0.0 1.0 -0.0"/>
   <limit upper="2.268928" lower="-2.268928" effort="100" velocity="100"/>
-</joint>
+</joint> -->
 </robot>

Commit message: manipulator model, ready

File: modelos/manipuladores/brazo_omni_v2_description/urdf/brazo_omni_v2.xacro (robot description, xacro)
@@ -104,24 +104,4 @@
   </collision>
 </link>
-<link name="eff1_1">
-  <inertial>
-    <origin xyz="0.00022190767864116318 -0.024999995073830102 0.0033250062490560728" rpy="0 0 0"/>
-    <mass value="0.23955016544085592"/>
-    <inertia ixx="7e-05" iyy="4.8e-05" izz="4.4e-05" ixy="0.0" iyz="-0.0" ixz="-2e-06"/>
-  </inertial>
-  <visual>
-    <origin xyz="-0.0 -0.025 -0.475" rpy="0 0 0"/>
-    <geometry>
-      <mesh filename="package://brazo_omni_v2_description/meshes/eff1_1.stl" scale="0.001 0.001 0.001"/>
-    </geometry>
-    <material name="silver"/>
-  </visual>
-  <collision>
-    <origin xyz="-0.0 -0.025 -0.475" rpy="0 0 0"/>
-    <geometry>
-      <mesh filename="package://brazo_omni_v2_description/meshes/eff1_1.stl" scale="0.001 0.001 0.001"/>
-    </geometry>
-  </collision>
-</link>
 <link name="eff2_1">
   <inertial>
@@ -140,5 +120,5 @@
     <origin xyz="-0.009226 0.0 -0.525981" rpy="0 0 0"/>
     <geometry>
-      <mesh filename="package://brazo_omni_v2_description/meshes/eff_2_1.stl" scale="0.001 0.001 0.001"/>
+      <mesh filename="package://brazo_omni_v2_description/meshes/eff2_1.stl" scale="0.001 0.001 0.001"/>
     </geometry>
   </collision>
@@ -156,5 +136,5 @@
   <child link="l2_1"/>
   <axis xyz="0.0 1.0 0.0"/>
-  <limit upper="1.989675" lower="-1.989675" effort="100" velocity="100"/>
+  <limit upper="1.919862" lower="-1.919862" effort="100" velocity="100"/>
 </joint>
 <joint name="l3_to_l2" type="revolute">
@@ -162,6 +142,6 @@
   <parent link="l2_1"/>
   <child link="l3_1"/>
-  <axis xyz="0.0 1.0 0.0"/>
-  <limit upper="1.989675" lower="-1.989675" effort="100" velocity="100"/>
+  <axis xyz="0.0 1.0 -0.0"/>
+  <limit upper="1.919862" lower="-1.919862" effort="100" velocity="100"/>
 </joint>
 <joint name="end_effector_to_l3" type="revolute">
@@ -169,11 +149,11 @@
   <parent link="l3_1"/>
   <child link="eff1_1"/>
-  <axis xyz="0.0 1.0 0.0"/>
+  <axis xyz="-0.0 1.0 -0.0"/>
   <limit upper="2.094395" lower="-2.094395" effort="100" velocity="100"/>
 </joint>
 <joint name="eff_2_to_eff_1" type="fixed">
   <origin xyz="0.009226 -0.025 0.050981" rpy="0 0 0"/>
-  <parent link="eff_1_1"/>
-  <child link="eff_2_1"/>
+  <parent link="eff1_1"/>
+  <child link="eff2_1"/>
 </joint>
 </robot>
