Commit message: base challenge

File: modelos/objetos/mini_bag_description/urdf/mini_bag.xacro (robot description, xacro)
@@ -15,5 +15,7 @@
       <mesh filename="package://mini_bag_description/meshes/base_link.stl" scale="0.001 0.001 0.001"/>
     </geometry>
-    <material name="silver"/>
+    <material name="pink">
+        <color rgba="255 0 132 0.9" />
+    </material>
   </visual>
   <collision concave="yes">
